Commit message: feat: implement Gazebo simulation setup for Speedpilot, including launch files and world configuration

File: ros2_ws/src/speedpilot_description/urdf/car.urdf.xacro (robot description, xacro)
@@ -1,21 +1,11 @@
 <?xml version="1.0"?>
 <robot xmlns:xacro="http://ros.org/wiki/xacro" name="speedpilot_car">
-  <!-- Material definitions -->
-  <material name="Blue">
-    <color rgba="0 0 1 1"/>
-  </material>
-  <material name="DarkGray">
-    <color rgba="0.3 0.3 0.3 1"/>
-  </material>
-  <material name="Black">
-    <color rgba="0 0 0 1"/>
-  </material>
-  <material name="Orange">
-    <color rgba="1 0.5 0 1"/>
-  </material>
-  <material name="Silver">
-    <color rgba="0.75 0.75 0.75 1"/>
-  </material>
-  <!-- Maße & Parameter -->
+  <!-- Materialien -->
+  <material name="Blue"><color rgba="0 0 1 1"/></material>
+  <material name="DarkGray"><color rgba="0.3 0.3 0.3 1"/></material>
+  <material name="Black"><color rgba="0 0 0 1"/></material>
+  <material name="Orange"><color rgba="1 0.5 0 1"/></material>
+  <material name="Silver"><color rgba="0.75 0.75 0.75 1"/></material>
+  <!-- Parameter -->
   <xacro:property name="wheel_radius" value="0.03"/>
   <xacro:property name="wheel_width" value="0.025"/>
@@ -26,62 +16,58 @@
   <xacro:property name="chassis_height_front" value="0.02"/>
   <xacro:property name="chassis_height_rear" value="0.07"/>
-  <xacro:property name="chassis_clearance" value="0.02"/> <!-- jetzt 2cm über Boden -->
+  <xacro:property name="chassis_clearance" value="0.02"/>
   <xacro:property name="lidar_height" value="0.12"/>
   <xacro:property name="ultrasound_height" value="0.025"/>
   <!-- Base Chassis -->
   <link name="base_link">
-    <!-- Vorderer Block -->
     <visual>
       <origin xyz="-0.0375 0 ${chassis_clearance + chassis_height_front / 2}" rpy="0 0 0"/>
-      <geometry>
-        <box size="${chassis_front_length} ${chassis_width_front} ${chassis_height_front}"/>
-      </geometry>
+      <geometry><box size="${chassis_front_length} ${chassis_width_front} ${chassis_height_front}"/></geometry>
       <material name="Blue"/>
     </visual>
-    <!-- Hinterer Block -->
     <visual>
       <origin xyz="-0.1875 0 ${chassis_clearance + chassis_height_rear / 2}" rpy="0 0 0"/>
-      <geometry>
-        <box size="${chassis_rear_length} ${chassis_width_rear} ${chassis_height_rear}"/>
-      </geometry>
+      <geometry><box size="${chassis_rear_length} ${chassis_width_rear} ${chassis_height_rear}"/></geometry>
       <material name="DarkGray"/>
     </visual>
+    <collision>
+      <origin xyz="-0.1 0 ${chassis_clearance + 0.035}" rpy="0 0 0"/>
+      <geometry><box size="0.3 0.1 0.1"/></geometry>
+    </collision>
+    <inertial>
+      <mass value="5.0"/>
+      <inertia ixx="0.1" iyy="0.1" izz="0.1" ixy="0.0" ixz="0.0" iyz="0.0"/>
+    </inertial>
   </link>
   <!-- LiDAR -->
   <link name="lidar_link">
     <visual>
-      <origin xyz="0.00 0 -0.008" rpy="0 0 0"/> <!-- Korrigierte Höhe -->
-      <geometry>
-        <cylinder radius="0.025" length="0.05"/>
-      </geometry>
+      <origin xyz="0.00 0 -0.008"/>
+      <geometry><cylinder radius="0.025" length="0.05"/></geometry>
       <material name="Black"/>
     </visual>
+    <collision>
+      <origin xyz="0.00 0 -0.008"/>
+      <geometry><cylinder radius="0.025" length="0.05"/></geometry>
+    </collision>
+    <inertial>
+      <mass value="0.1"/>
+      <inertia ixx="0.001" iyy="0.001" izz="0.001" ixy="0.0" ixz="0.0" iyz="0.0"/>
+    </inertial>
   </link>
   <joint name="lidar_joint" type="fixed">
     <parent link="base_link"/>
     <child link="lidar_link"/>
-    <origin xyz="-0.125 0 ${lidar_height}" rpy="0 0 0"/>
+    <origin xyz="-0.125 0 ${lidar_height}"/>
   </joint>
-  <!-- LiDAR Sensor Plugin -->
   <gazebo reference="lidar_link">
     <sensor type="ray" name="lidar_sensor">
       <update_rate>10.0</update_rate>
       <ray>
-        <scan>
-          <horizontal>
-            <samples>360</samples>
-            <min_angle>-3.14</min_angle>
-            <max_angle>3.14</max_angle>
-          </horizontal>
-        </scan>
-        <range>
-          <min>0.12</min>
-          <max>5.0</max>
-        </range>
+        <scan><horizontal><samples>360</samples><min_angle>-3.14</min_angle><max_angle>3.14</max_angle></horizontal></scan>
+        <range><min>0.12</min><max>5.0</max></range>
       </ray>
       <plugin name="gazebo_ros_laser_controller" filename="libgazebo_ros_ray_sensor.so">
-        <ros>
-          <remapping>~/scan:=scan</remapping>
-        </ros>
+        <ros><remapping>~/scan:=scan</remapping></ros>
       </plugin>
     </sensor>
@@ -90,31 +76,39 @@
   <link name="ultrasound_link">
     <visual>
-      <origin xyz="-0.0 0 0.02" rpy="0 0 0"/> <!-- keine Rotation nötig -->
-      <geometry>
-        <box size="0.015 0.055 ${ultrasound_height}"/> <!-- Länge in X -->
-      </geometry>
+      <origin xyz="0 0 0.02"/>
+      <geometry><box size="0.015 0.055 ${ultrasound_height}"/></geometry>
       <material name="Orange"/>
     </visual>
+    <inertial>
+      <mass value="0.05"/>
+      <inertia ixx="0.0001" iyy="0.0001" izz="0.0001" ixy="0.0" ixz="0.0" iyz="0.0"/>
+    </inertial>
   </link>
   <joint name="ultrasound_joint" type="fixed">
     <parent link="base_link"/>
     <child link="ultrasound_link"/>
-    <origin xyz="-0.01 0 0.03" rpy="0 0 0"/>
+    <origin xyz="-0.01 0 0.03"/>
   </joint>
-  <!-- Räder -->
+  <!-- Rad-Makro -->
   <xacro:macro name="wheel" params="name x y">
     <link name="${name}">
       <visual>
         <origin xyz="0 0 0" rpy="1.5708 0 0"/>
-        <geometry>
-          <cylinder radius="${wheel_radius}" length="${wheel_width}"/>
-        </geometry>
+        <geometry><cylinder radius="${wheel_radius}" length="${wheel_width}"/></geometry>
         <material name="Black"/>
       </visual>
+      <collision>
+        <origin xyz="0 0 0" rpy="1.5708 0 0"/>
+        <geometry><cylinder radius="${wheel_radius}" length="${wheel_width}"/></geometry>
+      </collision>
+      <inertial>
+        <mass value="0.2"/>
+        <inertia ixx="0.001" iyy="0.001" izz="0.001" ixy="0.0" ixz="0.0" iyz="0.0"/>
+      </inertial>
     </link>
     <joint name="${name}_joint" type="continuous">
       <parent link="base_link"/>
       <child link="${name}"/>
-      <origin xyz="${x} ${y} ${wheel_radius}" rpy="0 0 0"/>
+      <origin xyz="${x} ${y} ${wheel_radius}"/>
       <axis xyz="0 1 0"/>
     </joint>
@@ -128,5 +122,5 @@
     <parent link="base_link"/>
     <child link="left_steer_hinge"/>
-    <origin xyz="-0.125 0.075 ${wheel_radius}" rpy="0 0 0"/>
+    <origin xyz="-0.125 0.075 ${wheel_radius}"/>
     <axis xyz="0 0 1"/>
     <limit effort="1.0" lower="-0.2618" upper="0.2618" velocity="1.0"/>
@@ -136,5 +130,4 @@
     <parent link="left_steer_hinge"/>
     <child link="left_front_wheel"/>
-    <origin xyz="0 0 0" rpy="0 0 0"/>
   </joint>
   <link name="right_steer_hinge"/>
@@ -142,5 +135,5 @@
     <parent link="base_link"/>
     <child link="right_steer_hinge"/>
-    <origin xyz="-0.125 -0.075 ${wheel_radius}" rpy="0 0 0"/>
+    <origin xyz="-0.125 -0.075 ${wheel_radius}"/>
     <axis xyz="0 0 1"/>
     <limit effort="1.0" lower="-0.2618" upper="0.2618" velocity="1.0"/>
@@ -150,35 +143,52 @@
     <parent link="right_steer_hinge"/>
     <child link="right_front_wheel"/>
-    <origin xyz="0 0 0" rpy="0 0 0"/>
   </joint>
-<!-- Hintere Achse -->
-<link name="rear_axle_link">
-  <visual>
-    <origin xyz="0 0 0" rpy="1.5708 0 0"/> <!-- nur visuelle Rotation -->
-    <geometry>
-      <cylinder length="0.15" radius="0.005"/>
-    </geometry>
-    <material name="Silver"/>
-  </visual>
-</link>
-<joint name="rear_axle_joint" type="fixed">
-  <parent link="base_link"/>
-  <child link="rear_axle_link"/>
-  <origin xyz="-0.285 0 ${wheel_radius}" rpy="0 0 0"/> <!-- reine Positionierung -->
-</joint>
-<!-- Vordere Achse -->
-<link name="front_axle_link">
-  <visual>
-    <origin xyz="0 0 0" rpy="1.5708 0 0"/>
-    <geometry>
-      <cylinder length="0.15" radius="0.005"/>
-    </geometry>
-    <material name="Silver"/>
-  </visual>
-</link>
-<joint name="front_axle_joint" type="fixed">
-  <parent link="base_link"/>
-  <child link="front_axle_link"/>
-  <origin xyz="-0.125 0 ${wheel_radius}" rpy="0 0 0"/>
-</joint>
+  <!-- Achsen -->
+  <link name="rear_axle_link">
+    <visual>
+      <origin xyz="0 0 0" rpy="1.5708 0 0"/>
+      <geometry><cylinder length="0.15" radius="0.005"/></geometry>
+      <material name="Silver"/>
+    </visual>
+    <inertial>
+      <mass value="0.1"/>
+      <inertia ixx="0.0002" iyy="0.0002" izz="0.0002" ixy="0.0" ixz="0.0" iyz="0.0"/>
+    </inertial>
+  </link>
+  <joint name="rear_axle_joint" type="fixed">
+    <parent link="base_link"/>
+    <child link="rear_axle_link"/>
+    <origin xyz="-0.285 0 ${wheel_radius}"/>
+  </joint>
+  <link name="front_axle_link">
+    <visual>
+      <origin xyz="0 0 0" rpy="1.5708 0 0"/>
+      <geometry><cylinder length="0.15" radius="0.005"/></geometry>
+      <material name="Silver"/>
+    </visual>
+    <inertial>
+      <mass value="0.1"/>
+      <inertia ixx="0.0002" iyy="0.0002" izz="0.0002" ixy="0.0" ixz="0.0" iyz="0.0"/>
+    </inertial>
+  </link>
+  <joint name="front_axle_joint" type="fixed">
+    <parent link="base_link"/>
+    <child link="front_axle_link"/>
+    <origin xyz="-0.125 0 ${wheel_radius}"/>
+  </joint>
+  <!-- Gazebo DiffDrive Plugin -->
+  <gazebo>
+    <plugin name="diff_drive_controller" filename="libgazebo_ros_diff_drive.so">
+      <ros><remapping>cmd_vel:=cmd_vel</remapping></ros>
+      <leftJoint>left_rear_wheel_joint</leftJoint>
+      <rightJoint>right_rear_wheel_joint</rightJoint>
+      <wheelSeparation>0.15</wheelSeparation>
+      <wheelDiameter>0.06</wheelDiameter>
+      <commandTopic>cmd_vel</commandTopic>
+      <odometryTopic>odom</odometryTopic>
+      <odometryFrame>odom</odometryFrame>
+      <robotBaseFrame>base_link</robotBaseFrame>
+      <publishOdomTf>true</publishOdomTf>
+    </plugin>
+  </gazebo>
 </robot>
